File: leds.kicad_sch (KiCad schematic)
At the start: 0 parts

Commit message: Added oled hierarchical page and referenced other pages
Parts:
- added D? (x2): LED, LED_THT:LED_D2.0mm_W4.0mm_H2.8mm_FlatTop, symbol Device:LED
- added R?: 320, Resistor_SMD:R_0201_0603Metric, symbol Device:R
- added R?: 220, Resistor_SMD:R_0201_0603Metric, symbol Device:R
Connections:
- new net: D?.2 (A), R?.2 (x2)
- new net GND: D?.1 (K), D?.1 (K)
- new net LED1G: R?.1
- new net LED2R: R?.1
Other:
- note added: "LEDs"

Commit message: Annotated all components (numerating)
Parts:
- gave numbers to parts that had none: 4
Changed lines of the file:
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@@
 		(on_board yes)
 		(dnp no)
-		(property "Reference" "R?"
+		(property "Reference" "R31"
 			(at 54.61 59.69 90)
 			(effects
@@
 			(project "diggi_shield_2"
 				(path "/21684161-6457-4723-8fc3-25d7330779e2/bed406b6-12b0-4660-ab7b-74b01e005d7a"
-					(reference "R?")
+					(reference "R31")
 					(unit 1)
 				)
@@
 		(dnp no)
 		(fields_autoplaced yes)
-		(property "Reference" "D?"
+		(property "Reference" "D2"
 			(at 67.6275 58.42 0)
 			(effects
@@
 			(project "diggi_shield_2"
 				(path "/21684161-6457-4723-8fc3-25d7330779e2/bed406b6-12b0-4660-ab7b-74b01e005d7a"
-					(reference "D?")
+					(reference "D2")
 					(unit 1)
 				)
@@
 		(dnp no)
 		(fields_autoplaced yes)
-		(property "Reference" "D?"
+		(property "Reference" "D1"
 			(at 67.6275 41.91 0)
 			(effects
@@
 			(project "diggi_shield_2"
 				(path "/21684161-6457-4723-8fc3-25d7330779e2/bed406b6-12b0-4660-ab7b-74b01e005d7a"
-					(reference "D?")
+					(reference "D1")
 					(unit 1)
 				)
@@
 		(on_board yes)
 		(dnp no)
-		(property "Reference" "R?"
+		(property "Reference" "R30"
 			(at 54.61 43.18 90)
 			(effects
@@
 			(project "diggi_shield_2"
 				(path "/21684161-6457-4723-8fc3-25d7330779e2/bed406b6-12b0-4660-ab7b-74b01e005d7a"
-					(reference "R?")
-					(unit 1)
-				)
+					(reference "R30")
+					(unit 1)
+				)

Commit message: Solve all warnings
Changed lines of the file:
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@@
-	)
-	(junction
-		(at 69.85 78.74)
-		(diameter 0)
-		(color 0 0 0 0)
 	)
 	(junction
@@
 	(wire
 		(pts
-			(xy 69.85 49.53) (xy 69.85 66.04)
+			(xy 69.85 66.04) (xy 69.85 78.74)
 		)
 		(stroke
@@
 	(wire
 		(pts
-			(xy 69.85 78.74) (xy 69.85 80.01)
+			(xy 69.85 49.53) (xy 69.85 66.04)
 		)
 		(stroke
-			(width 0)
-			(type default)
-		)
-	)
-	(wire
-		(pts
-			(xy 69.85 66.04) (xy 69.85 78.74)
-		)
-		(stroke
