File: power.kicad_sch (KiCad schematic)
At the start: 0 parts

Commit message: Added oled hierarchical page and referenced other pages
Parts:
- added C? (x4): 47u, Capacitor_SMD:C_1206_3216Metric, symbol Device:C_Small
- added C? (x4): 100n, Capacitor_SMD:C_0603_1608Metric, symbol Device:C_Small
- added C? (x2): 10u, Capacitor_SMD:C_0603_1608Metric, symbol Device:C_Small
- added C?: 10n, Capacitor_SMD:C_0603_1608Metric, symbol Device:C_Small
- added D?: 3V3, Diode_SMD:D_MiniMELF, symbol Device:D_Zener
- added D? (x2): SS34, Diode_SMD:D_SMA, symbol Diode:1N5819
- added D?: LED, LED_SMD:LED_0603_1608Metric, symbol Device:LED
- added J?: DC 9-20V, Connector_BarrelJack:BarrelJack_GCT_DCJ200-10-A_Horizontal, symbol Connector:Barrel_Jack_Switch
- added J?: VIN, Connector_PinHeader_2.54mm:PinHeader_1x02_P2.54mm_Vertical, symbol Connector:Conn_01x02_Male
- added L?: 15uh, Inductor_SMD:L_10.4x10.4_H4.8, symbol pspice:INDUCTOR
- added R?: 3k, Resistor_SMD:R_0603_1608Metric, symbol Device:R
- added R? (x2): 10k, Resistor_SMD:R_0603_1608Metric, symbol Device:R
- added R?: 47k, Resistor_SMD:R_0603_1608Metric, symbol Device:R
- added R?: 220, Resistor_SMD:R_0603_1608Metric, symbol Device:R
- added U?: 74HC14, Package_SO:SOIC-14_3.9x8.7mm_P1.27mm, symbol 74xx:74HC14
- added U?: TPS5430DDA, Package_SO:TI_SO-PowerPAD-8_ThermalVias, symbol Regulator_Switching:TPS5430DDA
Connections:
- new net: D?.2 (A), J?.1, J?.1 (Pin_1), R?.2
- new net: C?.1, C?.1, C?.1, D?.1 (K), U?.7 (VIN)
- new net: C?.1, D?.1 (K), L?.1, U?.8 (PH)
- new net: R?.1, R?.2
- new net: R?.2, R?.2, U?.4 (VSENSE)
- new net: D?.2 (A), R?.2
- new net: C?.2, U?.1 (BOOT)
- new net +5V: C?.1, C?.1, C?.1, C?.1, C?.1, C?.1, L?.2, R?.1, R?.1
- new net GND: C?.2, C?.2, C?.2, C?.2, C?.2, C?.2, C?.2, C?.2, C?.2, C?.2, D?.1 (K), D?.2 (A), D?.2 (A), J?.2, J?.2 (Pin_2), R?.1, U?.6 (GND), U?.9 (GNDPAD)
- new net VBUS_END: C?.1, D?.1 (K), R?.1, U?.5 (EN)
- no-connect marks 0 -> 1
Other:
- note added: "DC to 5V"
- note added: "R2 = (R1*1.221) / (Vout - 1.221) = (10000*1.221) / (5 - 1.221) = 12210 / 3,779 R2 = 3231 ohm"
- note added: "ceramic preferred"
- note added: "power lamp"

Commit message: Fixed pcb and ran some electrical rule checking and fixed some issues mainly connections and power flags
Changed lines of the file:
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@@
 	)
 	(junction
-		(at 44.45 59.69)
-		(diameter 0)
-		(color 0 0 0 0)
-	)
-	(junction
 		(at 149.86 59.69)
 		(diameter 0)
@@
 		(color 0 0 0 0)
 	)
-	(junction
-		(at 184.15 57.15)
-		(diameter 0)
-		(color 0 0 0 0)
-	)
 	(no_connect
 		(at 44.45 57.15)
@@
 		(on_board yes)
 		(dnp no)
-		(property "Reference" "#PWR?"
+		(property "Reference" "#PWR0251"
 			(at 44.45 66.04 0)
 			(effects
@@
 			(project "diggi_shield_2"
 				(path "/21684161-6457-4723-8fc3-25d7330779e2/788df4b9-9107-41b0-b5cb-b766128c8ce8"
-					(reference "#PWR?")
+					(reference "#PWR0251")
 					(unit 1)
 				)
@@
 		(dnp no)
 		(fields_autoplaced yes)
-		(property "Reference" "#PWR?"
+		(property "Reference" "#PWR0266"
 			(at 62.23 114.3 0)
 			(effects
@@
 			(project "diggi_shield_2"
 				(path "/21684161-6457-4723-8fc3-25d7330779e2/788df4b9-9107-41b0-b5cb-b766128c8ce8"
-					(reference "#PWR?")
+					(reference "#PWR0266")
 					(unit 1)
 				)
@@
 		(dnp no)
 		(fields_autoplaced yes)
-		(property "Reference" "#PWR?"
+		(property "Reference" "#PWR0263"
 			(at 204.47 102.87 0)
 			(effects
@@
 			(project "diggi_shield_2"
 				(path "/21684161-6457-4723-8fc3-25d7330779e2/788df4b9-9107-41b0-b5cb-b766128c8ce8"
-					(reference "#PWR?")
+					(reference "#PWR0263")
 					(unit 1)
 				)
@@
 		(on_board yes)
 		(dnp no)
-		(property "Reference" "#PWR?"
+		(property "Reference" "#PWR0264"
 			(at 184.15 71.12 0)
 			(effects
@@
 			(project "diggi_shield_2"
 				(path "/21684161-6457-4723-8fc3-25d7330779e2/788df4b9-9107-41b0-b5cb-b766128c8ce8"
-					(reference "#PWR?")
+					(reference "#PWR0264")
 					(unit 1)
 				)
@@
 		(on_board yes)
 		(dnp no)
-		(property "Reference" "#PWR?"
+		(property "Reference" "#PWR0254"
 			(at 135.89 74.93 0)
 			(effects
@@
 			(project "diggi_shield_2"
 				(path "/21684161-6457-4723-8fc3-25d7330779e2/788df4b9-9107-41b0-b5cb-b766128c8ce8"
-					(reference "#PWR?")
+					(reference "#PWR0254")
 					(unit 1)
 				)
@@
 		(on_board yes)
 		(dnp no)
-		(property "Reference" "#PWR?"
+		(property "Reference" "#PWR0255"
 			(at 114.3 76.2 0)
 			(effects
@@
 			(project "diggi_shield_2"
 				(path "/21684161-6457-4723-8fc3-25d7330779e2/788df4b9-9107-41b0-b5cb-b766128c8ce8"
-					(reference "#PWR?")
+					(reference "#PWR0255")
 					(unit 1)
 				)
@@
 		(on_board yes)
 		(dnp no)
-		(property "Reference" "#PWR?"
+		(property "Reference" "#PWR0257"
 			(at 165.1 71.12 0)
 			(effects
@@
 			(project "diggi_shield_2"
 				(path "/21684161-6457-4723-8fc3-25d7330779e2/788df4b9-9107-41b0-b5cb-b766128c8ce8"
-					(reference "#PWR?")
+					(reference "#PWR0257")
 					(unit 1)
 				)
@@
 		(on_board yes)
 		(dnp no)
-		(property "Reference" "#PWR?"
+		(property "Reference" "#PWR0267"
 			(at 68.58 90.17 0)
 			(effects
@@
 			(project "diggi_shield_2"
 				(path "/21684161-6457-4723-8fc3-25d7330779e2/788df4b9-9107-41b0-b5cb-b766128c8ce8"
-					(reference "#PWR?")
+					(reference "#PWR0267")
 					(unit 1)
 				)
@@
 		(on_board yes)
 		(dnp no)
-		(property "Reference" "#PWR?"
+		(property "Reference" "#PWR0256"
 			(at 157.48 71.12 0)
 			(effects
@@
 			(project "diggi_shield_2"
 				(path "/21684161-6457-4723-8fc3-25d7330779e2/788df4b9-9107-41b0-b5cb-b766128c8ce8"
-					(reference "#PWR?")
+					(reference "#PWR0256")
 					(unit 1)
 				)
@@
 		(on_board yes)
 		(dnp no)
-		(property "Reference" "#PWR?"
+		(property "Reference" "#PWR0262"
 			(at 193.04 71.12 0)
 			(effects
@@
 			(project "diggi_shield_2"
 				(path "/21684161-6457-4723-8fc3-25d7330779e2/788df4b9-9107-41b0-b5cb-b766128c8ce8"
-					(reference "#PWR?")
+					(reference "#PWR0262")
 					(unit 1)
 				)
@@
 		(dnp no)
 		(fields_autoplaced yes)
-		(property "Reference" "#PWR?"
+		(property "Reference" "#PWR0258"
 			(at 208.28 110.49 0)
 			(effects
@@
 			(project "diggi_shield_2"
 				(path "/21684161-6457-4723-8fc3-25d7330779e2/788df4b9-9107-41b0-b5cb-b766128c8ce8"
-					(reference "#PWR?")
+					(reference "#PWR0258")
 					(unit 1)
 				)
@@
 		(dnp no)
 		(fields_autoplaced yes)
-		(property "Reference" "#PWR?"
+		(property "Reference" "#PWR0259"
 			(at 204.47 137.16 0)
 			(effects
@@
 			(project "diggi_shield_2"
 				(path "/21684161-6457-4723-8fc3-25d7330779e2/788df4b9-9107-41b0-b5cb-b766128c8ce8"
-					(reference "#PWR?")
+					(reference "#PWR0259")
 					(unit 1)
 				)
@@
 		(on_board yes)
 		(dnp no)
-		(property "Reference" "#PWR?"
+		(property "Reference" "#PWR0249"
 			(at 54.61 63.5 0)
 			(effects
@@
 			(project "diggi_shield_2"
 				(path "/21684161-6457-4723-8fc3-25d7330779e2/788df4b9-9107-41b0-b5cb-b766128c8ce8"
-					(reference "#PWR?")
+					(reference "#PWR0249")
 					(unit 1)
 				)
@@
 	(symbol
 		(lib_id "power:PWR_FLAG")
-		(at 44.45 59.69 270)
-		(unit 1)
-		(exclude_from_sim no)
-		(in_bom yes)
-		(on_board yes)
-		(dnp no)
-		(fields_autoplaced yes)
-		(property "Reference" "#FLG?"
-			(at 46.355 59.69 0)
-			(effects
-				(font
-					(size 1.27 1.27)
-				)
-				(hide yes)
-			)
-		)
-		(property "Value" "PWR_FLAG"
-			(at 48.26 59.69 0)
-			(effects
-				(font
-					(size 1.27 1.27)
-				)
-				(hide yes)
-			)
-		)
-		(property "Footprint" ""
-			(at 44.45 59.69 0)
-			(effects
-				(font
-					(size 1.27 1.27)
-				)
-				(hide yes)
-			)
-		)
-		(property "Datasheet" "~"
-			(at 44.45 59.69 0)
-			(effects
-				(font
-					(size 1.27 1.27)
-				)
-				(hide yes)
-			)
-		)
-		(property "Description" ""
-			(at 44.45 59.69 0)
-			(effects
-				(font
-					(size 1.27 1.27)
-				)
-				(hide yes)
-			)
-		)
-		(pin "1"
-		)
-		(instances
-			(project "diggi_shield_2"
-				(path "/21684161-6457-4723-8fc3-25d7330779e2/788df4b9-9107-41b0-b5cb-b766128c8ce8"
-					(reference "#FLG?")
-					(unit 1)
-				)
-			)
-		)
-	)
-	(symbol
-		(lib_id "power:PWR_FLAG")
 		(at 97.79 54.61 0)
 		(unit 1)
@@
 		(dnp no)
 		(fields_autoplaced yes)
-		(property "Reference" "#FLG?"
+		(property "Reference" "#FLG0101"
 			(at 97.79 52.705 0)
 			(effects
@@
 			(project "diggi_shield_2"
 				(path "/21684161-6457-4723-8fc3-25d7330779e2/788df4b9-9107-41b0-b5cb-b766128c8ce8"
-					(reference "#FLG?")
+					(reference "#FLG0101")
 					(unit 1)
 				)
@@
 		(on_board yes)
 		(dnp no)
-		(property "Reference" "#PWR?"
+		(property "Reference" "#PWR0250"
 			(at 85.09 67.31 0)
 			(effects
@@
 			(project "diggi_shield_2"
 				(path "/21684161-6457-4723-8fc3-25d7330779e2/788df4b9-9107-41b0-b5cb-b766128c8ce8"
-					(reference "#PWR?")
+					(reference "#PWR0250")
 					(unit 1)
 				)
@@
 		(dnp no)
 		(fields_autoplaced yes)
-		(property "Reference" "#PWR?"
+		(property "Reference" "#PWR0260"
 			(at 184.15 60.96 0)
 			(effects
@@
 			(project "diggi_shield_2"
 				(path "/21684161-6457-4723-8fc3-25d7330779e2/788df4b9-9107-41b0-b5cb-b766128c8ce8"
-					(reference "#PWR?")
+					(reference "#PWR0260")
 					(unit 1)
 				)
@@
 		(on_board yes)
 		(dnp no)
-		(property "Reference" "#PWR?"
+		(property "Reference" "#PWR0253"
 			(at 149.86 88.9 0)
 			(effects
@@
 			(project "diggi_shield_2"
 				(path "/21684161-6457-4723-8fc3-25d7330779e2/788df4b9-9107-41b0-b5cb-b766128c8ce8"
-					(reference "#PWR?")
+					(reference "#PWR0253")
 					(unit 1)
 				)
@@
 		(on_board yes)
 		(dnp no)
-		(property "Reference" "#PWR?"
+		(property "Reference" "#PWR0269"
 			(at 62.23 132.08 0)
 			(effects
@@
 			(project "diggi_shield_2"
 				(path "/21684161-6457-4723-8fc3-25d7330779e2/788df4b9-9107-41b0-b5cb-b766128c8ce8"
-					(reference "#PWR?")
+					(reference "#PWR0269")
 					(unit 1)
 				)
@@
 		(on_board yes)
 		(dnp no)
-		(property "Reference" "#PWR?"
+		(property "Reference" "#PWR0265"
 			(at 76.2 67.31 0)
 			(effects
@@
 			(project "diggi_shield_2"
 				(path "/21684161-6457-4723-8fc3-25d7330779e2/788df4b9-9107-41b0-b5cb-b766128c8ce8"
-					(reference "#PWR?")
+					(reference "#PWR0265")
 					(unit 1)
 				)
@@
 		(on_board yes)
 		(dnp no)
-		(property "Reference" "#PWR?"
+		(property "Reference" "#PWR0252"
 			(at 97.79 67.31 0)
 			(effects
@@
 			(project "diggi_shield_2"
 				(path "/21684161-6457-4723-8fc3-25d7330779e2/788df4b9-9107-41b0-b5cb-b766128c8ce8"
-					(reference "#PWR?")
+					(reference "#PWR0252")
 					(unit 1)
 				)
@@
 	)
 	(symbol
-		(lib_id "power:PWR_FLAG")
-		(at 184.15 57.15 270)
-		(unit 1)
-		(exclude_from_sim no)
-		(in_bom yes)
-		(on_board yes)
-		(dnp no)
-		(fields_autoplaced yes)
-		(property "Reference" "#FLG?"
-			(at 186.055 57.15 0)
-			(effects
-				(font
-					(size 1.27 1.27)
-				)
-				(hide yes)
-			)
-		)
-		(property "Value" "PWR_FLAG"
-			(at 187.96 57.15 0)
-			(effects
-				(font
-					(size 1.27 1.27)
-				)
-				(hide yes)
-			)
-		)
-		(property "Footprint" ""
-			(at 184.15 57.15 0)
-			(effects
-				(font
-					(size 1.27 1.27)
-				)
-				(hide yes)
-			)
-		)
-		(property "Datasheet" "~"
-			(at 184.15 57.15 0)
-			(effects
-				(font
-					(size 1.27 1.27)
-				)
-				(hide yes)
-			)
-		)
-		(property "Description" ""
-			(at 184.15 57.15 0)
-			(effects
-				(font
-					(size 1.27 1.27)
-				)
-				(hide yes)
-			)
-		)
-		(pin "1"
-		)
-		(instances
-			(project "diggi_shield_2"
-				(path "/21684161-6457-4723-8fc3-25d7330779e2/788df4b9-9107-41b0-b5cb-b766128c8ce8"
-					(reference "#FLG?")
-					(unit 1)
-				)
-			)
-		)
-	)
-	(symbol
 		(lib_id "Device:C_Small")
 		(at 184.15 62.23 0)
@@
 		(on_board yes)
 		(dnp no)
-		(property "Reference" "#PWR?"
+		(property "Reference" "#PWR0268"
 			(at 62.23 90.17 0)
 			(effects
@@
 			(project "diggi_shield_2"
 				(path "/21684161-6457-4723-8fc3-25d7330779e2/788df4b9-9107-41b0-b5cb-b766128c8ce8"
-					(reference "#PWR?")
+					(reference "#PWR0268")
 					(unit 1)
 				)
@@
 		(on_board yes)
 		(dnp no)
-		(property "Reference" "#PWR?"
+		(property "Reference" "#PWR0261"
 			(at 173.99 71.12 0)
 			(effects
@@
 			(project "diggi_shield_2"
 				(path "/21684161-6457-4723-8fc3-25d7330779e2/788df4b9-9107-41b0-b5cb-b766128c8ce8"
-					(reference "#PWR?")
+					(reference "#PWR0261")
 					(unit 1)
 				)

Commit message: Annotated all components (numerating)
Parts:
- gave numbers to parts that had none: 25
Changed lines of the file:
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@@
 		(dnp no)
 		(fields_autoplaced yes)
-		(property "Reference" "U?"
+		(property "Reference" "U7"
 			(at 210.82 116.8399 0)
 			(effects
@@
 			(project "diggi_shield_2"
 				(path "/21684161-6457-4723-8fc3-25d7330779e2/788df4b9-9107-41b0-b5cb-b766128c8ce8"
-					(reference "U?")
+					(reference "U7")
 					(unit 1)
 				)
@@
 		(on_board yes)
 		(dnp no)
-		(property "Reference" "J?"
+		(property "Reference" "J_PWR1"
 			(at 36.83 48.26 0)
 			(effects
@@
 			(project "diggi_shield_2"
 				(path "/21684161-6457-4723-8fc3-25d7330779e2/788df4b9-9107-41b0-b5cb-b766128c8ce8"
-					(reference "J?")
+					(reference "J_PWR1")
 					(unit 1)
 				)
@@
 		(on_board yes)
 		(dnp no)
-		(property "Reference" "C?"
+		(property "Reference" "C57"
 			(at 195.3768 61.0616 0)
 			(effects
@@
 			(project "diggi_shield_2"
 				(path "/21684161-6457-4723-8fc3-25d7330779e2/788df4b9-9107-41b0-b5cb-b766128c8ce8"
-					(reference "C?")
+					(reference "C57")
 					(unit 1)
 				)
@@
 		(on_board yes)
 		(dnp no)
-		(property "Reference" "C?"
+		(property "Reference" "C51"
 			(at 100.1268 55.9816 0)
 			(effects
@@
 			(project "diggi_shield_2"
 				(path "/21684161-6457-4723-8fc3-25d7330779e2/788df4b9-9107-41b0-b5cb-b766128c8ce8"
-					(reference "C?")
+					(reference "C51")
 					(unit 1)
 				)
@@
 		(dnp no)
 		(fields_autoplaced yes)
-		(property "Reference" "L?"
+		(property "Reference" "L1"
 			(at 143.51 54.8472 0)
 			(effects
@@
 			(project "diggi_shield_2"
 				(path "/21684161-6457-4723-8fc3-25d7330779e2/788df4b9-9107-41b0-b5cb-b766128c8ce8"
-					(reference "L?")
+					(reference "L1")
 					(unit 1)
 				)
@@
 		(dnp no)
 		(fields_autoplaced yes)
-		(property "Reference" "J?"
+		(property "Reference" "J2"
 			(at 50.165 49.53 0)
 			(effects
@@
 			(project "diggi_shield_2"
 				(path "/21684161-6457-4723-8fc3-25d7330779e2/788df4b9-9107-41b0-b5cb-b766128c8ce8"
-					(reference "J?")
+					(reference "J2")
 					(unit 1)
 				)
@@
 		(on_board yes)
 		(dnp no)
-		(property "Reference" "C?"
+		(property "Reference" "C49"
 			(at 78.5368 55.9816 0)
 			(effects
@@
 			(project "diggi_shield_2"
 				(path "/21684161-6457-4723-8fc3-25d7330779e2/788df4b9-9107-41b0-b5cb-b766128c8ce8"
-					(reference "C?")
+					(reference "C49")
 					(unit 1)
 				)
@@
 		(on_board yes)
 		(dnp no)
-		(property "Reference" "C?"
+		(property "Reference" "C50"
 			(at 87.4268 55.9816 0)
 			(effects
@@
 			(project "diggi_shield_2"
 				(path "/21684161-6457-4723-8fc3-25d7330779e2/788df4b9-9107-41b0-b5cb-b766128c8ce8"
-					(reference "C?")
+					(reference "C50")
 					(unit 1)
 				)
@@
 		(on_board yes)
 		(dnp no)
-		(property "Reference" "R?"
+		(property "Reference" "R52"
 			(at 151.638 77.9053 0)
 			(effects
@@
 			(project "diggi_shield_2"
 				(path "/21684161-6457-4723-8fc3-25d7330779e2/788df4b9-9107-41b0-b5cb-b766128c8ce8"
-					(reference "R?")
+					(reference "R52")
 					(unit 1)
 				)
@@
 		(dnp no)
 		(fields_autoplaced yes)
-		(property "Reference" "D?"
+		(property "Reference" "D6"
 			(at 71.12 74.9299 90)
 			(effects
@@
 			(project "diggi_shield_2"
 				(path "/21684161-6457-4723-8fc3-25d7330779e2/788df4b9-9107-41b0-b5cb-b766128c8ce8"
-					(reference "D?")
+					(reference "D6")
 					(unit 1)
 				)
@@
 		(dnp no)
 		(fields_autoplaced yes)
-		(property "Reference" "D?"
+		(property "Reference" "D7"
 			(at 138.43 63.1824 90)
 			(effects
@@
 			(project "diggi_shield_2"
 				(path "/21684161-6457-4723-8fc3-25d7330779e2/788df4b9-9107-41b0-b5cb-b766128c8ce8"
-					(reference "D?")
+					(reference "D7")
 					(unit 1)
 				)
@@
 		(on_board yes)
 		(dnp no)
-		(property "Reference" "R?"
+		(property "Reference" "R50"
 			(at 151.638 62.6653 0)
 			(effects
@@
 			(project "diggi_shield_2"
 				(path "/21684161-6457-4723-8fc3-25d7330779e2/788df4b9-9107-41b0-b5cb-b766128c8ce8"
-					(reference "R?")
+					(reference "R50")
 					(unit 1)
 				)
@@
 		(on_board yes)
 		(dnp no)
-		(property "Reference" "R?"
+		(property "Reference" "R49"
 			(at 64.008 113.4653 0)
 			(effects
@@
 			(project "diggi_shield_2"
 				(path "/21684161-6457-4723-8fc3-25d7330779e2/788df4b9-9107-41b0-b5cb-b766128c8ce8"
-					(reference "R?")
+					(reference "R49")
 					(unit 1)
 				)
@@
 		(on_board yes)
 		(dnp no)
-		(property "Reference" "C?"
+		(property "Reference" "C54"
 			(at 167.4368 61.0616 0)
 			(effects
@@
 			(project "diggi_shield_2"
 				(path "/21684161-6457-4723-8fc3-25d7330779e2/788df4b9-9107-41b0-b5cb-b766128c8ce8"
-					(reference "C?")
+					(reference "C54")
 					(unit 1)
 				)
@@
 		(dnp no)
 		(fields_autoplaced yes)
-		(property "Reference" "D?"
+		(property "Reference" "D5"
 			(at 66.3575 48.26 0)
 			(effects
@@
 			(project "diggi_shield_2"
 				(path "/21684161-6457-4723-8fc3-25d7330779e2/788df4b9-9107-41b0-b5cb-b766128c8ce8"
-					(reference "D?")
+					(reference "D5")
 					(unit 1)
 				)
@@
 		(on_board yes)
 		(dnp no)
-		(property "Reference" "C?"
+		(property "Reference" "C52"
 			(at 135.89 55.6514 0)
 			(effects
@@
 			(project "diggi_shield_2"
 				(path "/21684161-6457-4723-8fc3-25d7330779e2/788df4b9-9107-41b0-b5cb-b766128c8ce8"
-					(reference "C?")
+					(reference "C52")
 					(unit 1)
 				)
@@
 		(on_board yes)
 		(dnp no)
-		(property "Reference" "C?"
+		(property "Reference" "C55"
 			(at 176.3268 61.0616 0)
 			(effects
@@
 			(project "diggi_shield_2"
 				(path "/21684161-6457-4723-8fc3-25d7330779e2/788df4b9-9107-41b0-b5cb-b766128c8ce8"
-					(reference "C?")
+					(reference "C55")
 					(unit 1)
 				)
@@
 		(on_board yes)
 		(dnp no)
-		(property "Reference" "R?"
+		(property "Reference" "R48"
 			(at 64.008 63.9353 0)
 			(effects
@@
 			(project "diggi_shield_2"
 				(path "/21684161-6457-4723-8fc3-25d7330779e2/788df4b9-9107-41b0-b5cb-b766128c8ce8"
-					(reference "R?")
+					(reference "R48")
 					(unit 1)
 				)
@@
 		(on_board yes)
 		(dnp no)
-		(property "Reference" "R?"
+		(property "Reference" "R51"
 			(at 151.638 70.2853 0)
 			(effects
@@
 			(project "diggi_shield_2"
 				(path "/21684161-6457-4723-8fc3-25d7330779e2/788df4b9-9107-41b0-b5cb-b766128c8ce8"
-					(reference "R?")
+					(reference "R51")
 					(unit 1)
 				)
@@
 		(on_board yes)
 		(dnp no)
-		(property "Reference" "C?"
+		(property "Reference" "C53"
 			(at 159.8168 61.0616 0)
 			(effects
@@
 			(project "diggi_shield_2"
 				(path "/21684161-6457-4723-8fc3-25d7330779e2/788df4b9-9107-41b0-b5cb-b766128c8ce8"
-					(reference "C?")
+					(reference "C53")
 					(unit 1)
 				)
@@
 		(on_board yes)
 		(dnp no)
-		(property "Reference" "C?"
+		(property "Reference" "C48"
 			(at 55.245 74.295 0)
 			(effects
@@
 			(project "diggi_shield_2"
 				(path "/21684161-6457-4723-8fc3-25d7330779e2/788df4b9-9107-41b0-b5cb-b766128c8ce8"
-					(reference "C?")
+					(reference "C48")
 					(unit 1)
 				)
@@
 		(on_board yes)
 		(dnp no)
-		(property "Reference" "C?"
+		(property "Reference" "C58"
 			(at 210.6168 100.4316 0)
 			(effects
@@
 			(project "diggi_shield_2"
 				(path "/21684161-6457-4723-8fc3-25d7330779e2/788df4b9-9107-41b0-b5cb-b766128c8ce8"
-					(reference "C?")
+					(reference "C58")
 					(unit 1)
 				)
@@
 		(on_board yes)
 		(dnp no)
-		(property "Reference" "C?"
+		(property "Reference" "C56"
 			(at 186.4868 61.0616 0)
 			(effects
@@
 			(project "diggi_shield_2"
 				(path "/21684161-6457-4723-8fc3-25d7330779e2/788df4b9-9107-41b0-b5cb-b766128c8ce8"
-					(reference "C?")
+					(reference "C56")
 					(unit 1)
 				)
@@
 		(dnp no)
 		(fields_autoplaced yes)
-		(property "Reference" "D?"
+		(property "Reference" "D4"
 			(at 65.151 122.6728 90)
 			(effects
@@
 			(project "diggi_shield_2"
 				(path "/21684161-6457-4723-8fc3-25d7330779e2/788df4b9-9107-41b0-b5cb-b766128c8ce8"
-					(reference "D?")
+					(reference "D4")
 					(unit 1)
 				)
@@
 		(dnp no)
 		(fields_autoplaced yes)
-		(property "Reference" "U?"
+		(property "Reference" "U6"
 			(at 116.84 46.99 0)
 			(effects
@@
 			(project "diggi_shield_2"
 				(path "/21684161-6457-4723-8fc3-25d7330779e2/788df4b9-9107-41b0-b5cb-b766128c8ce8"
-					(reference "U?")
+					(reference "U6")
 					(unit 1)
 				)

Commit message: Cleaned up ERC errors
Parts:
- removed C58: 100n, Capacitor_SMD:C_0603_1608Metric, symbol Device:C_Small
- removed U7: 74HC14, Package_SO:SOIC-14_3.9x8.7mm_P1.27mm, symbol 74xx:74HC14

Commit message: Solve all warnings
Parts:
- J2: symbol Connector:Conn_01x02_Male -> Connector:Conn_01x02_Pin
- L1: symbol pspice:INDUCTOR -> Device:L
Changed lines of the file:
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@@
+	)
+	(junction
+		(at 149.86 59.69)
+		(diameter 0)
+		(color 0 0 0 0)
 	)
 	(junction
@@
 	)
 	(junction
-		(at 149.86 59.69)
-		(diameter 0)
-		(color 0 0 0 0)
-	)
-	(junction
 		(at 114.3 69.85)
 		(diameter 0)
@@
 	(wire
 		(pts
-			(xy 135.89 59.69) (xy 137.16 59.69)
+			(xy 135.89 59.69) (xy 139.7 59.69)
 		)
 		(stroke
@@
 		(pts
 			(xy 132.08 59.69) (xy 129.54 59.69)
+		)
+		(stroke
+			(width 0)
+			(type default)
+		)
+	)
+	(wire
+		(pts
+			(xy 147.32 59.69) (xy 149.86 59.69)
 		)
 		(stroke
@@
 	)
 	(symbol
-		(lib_id "pspice:INDUCTOR")
-		(at 143.51 59.69 0)
+		(lib_id "Device:L")
+		(at 143.51 59.69 90)
 		(unit 1)
 		(exclude_from_sim no)
@@
 		(fields_autoplaced yes)
 		(property "Reference" "L1"
-			(at 143.51 54.8472 0)
+			(at 143.51 54.61 90)
 			(effects
 				(font
@@
 		)
 		(property "Value" "15uh"
-			(at 143.51 57.3841 0)
+			(at 143.51 57.15 90)
 			(effects
 				(font
@@
 			)
 		)
-		(property "Description" ""
+		(property "Description" "Inductor"
 			(at 143.51 59.69 0)
 			(effects
@@
 	)
 	(symbol
-		(lib_id "Connector:Conn_01x02_Male")
+		(lib_id "Connector:Conn_01x02_Pin")
 		(at 49.53 54.61 0)
 		(unit 1)
@@
 			)
 		)
-		(property "Description" ""
+		(property "Description" "Generic connector, single row, 01x02, script generated"
 			(at 49.53 54.61 0)
 			(effects
