File: shiftregisters.kicad_sch (KiCad schematic)
At the start: 0 parts

Commit message: Added oled hierarchical page and referenced other pages
Parts:
- added C? (x5): 100nf, symbol Device:C_Small
- added U? (x5): 74HC165, symbol 74xx:74HC165
Connections:
- new net: U?.10 (DS), U?.9 (Q7) (x4)
- new net: C?.2, U?.16 (VCC) (x5)
- new net +3.3V: C?.1, C?.1, C?.1, C?.1, C?.1
- new net ENC1_A: U?.11 (D0)
- new net ENC1_B: U?.12 (D1)
- new net ENC1_SW: U?.13 (D2)
- new net ENC2_A: U?.11 (D0)
- new net ENC2_B: U?.12 (D1)
- new net ENC2_SW: U?.14 (D3)
- new net ENC3_A: U?.13 (D2)
- new net ENC3_B: U?.14 (D3)
- new net ENC3_SW: U?.3 (D4)
- new net ENC4_A: U?.3 (D4)
- new net ENC4_B: U?.4 (D5)
- new net ENC4_SW: U?.5 (D6)
- new net ENC5_A: U?.4 (D5)
- new net ENC5_B: U?.5 (D6)
- new net ENC5_SW: U?.6 (D7)
- new net ENC6_A: U?.4 (D5)
- new net ENC6_B: U?.5 (D6)
- new net ENC6_SW: U?.6 (D7)
- new net ENC7_A: U?.11 (D0)
- new net ENC7_B: U?.12 (D1)
- new net ENC7_SW: U?.13 (D2)
- new net ENC8_A: U?.14 (D3)
- new net ENC8_B: U?.3 (D4)
- new net ENC8_SW: U?.4 (D5)
- new net ENC9_A: U?.11 (D0)
- new net ENC9_B: U?.12 (D1)
- new net ENC9_SW: U?.13 (D2)
- new net GND: U?.15 (~{CE}), U?.15 (~{CE}), U?.15 (~{CE}), U?.15 (~{CE}), U?.15 (~{CE}), U?.8 (GND), U?.8 (GND)
- new net PA4: U?.1 (~{PL}), U?.1 (~{PL}), U?.1 (~{PL}), U?.1 (~{PL}), U?.1 (~{PL})
- new net PA5: U?.2 (CP), U?.2 (CP), U?.2 (CP), U?.2 (CP), U?.2 (CP)
- new net PA6: U?.9 (Q7)
- new net SW_1: U?.14 (D3)
- new net SW_2: U?.3 (D4)
- new net SW_3: U?.4 (D5)
- new net SW_4: U?.5 (D6)
- new net SW_5: U?.11 (D0)
- new net SW_6: U?.12 (D1)
- new net SW_7: U?.13 (D2)
- new net SW_8: U?.14 (D3)
- new net SW_A: U?.6 (D7)
- new net SW_B: U?.3 (D4)
- new net SW_C: U?.6 (D7)
- new net SW_D: U?.5 (D6)
- no-connect marks 0 -> 1

Commit message: Annotated all components (numerating)
Parts:
- gave numbers to parts that had none: 10
Changed lines of the file:
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@@
 		(dnp no)
 		(fields_autoplaced yes)
-		(property "Reference" "U?"
+		(property "Reference" "U2"
 			(at 103.7941 41.91 0)
 			(effects
@@
 			(project "diggi_shield_2"
 				(path "/21684161-6457-4723-8fc3-25d7330779e2/4a4e12e0-86da-4c7e-aa92-3e2740ba45ee"
-					(reference "U?")
+					(reference "U2")
 					(unit 1)
 				)
@@
 		(dnp no)
 		(fields_autoplaced yes)
-		(property "Reference" "C?"
+		(property "Reference" "C29"
 			(at 62.23 36.8362 0)
 			(effects
@@
 			(project "diggi_shield_2"
 				(path "/21684161-6457-4723-8fc3-25d7330779e2/4a4e12e0-86da-4c7e-aa92-3e2740ba45ee"
-					(reference "C?")
+					(reference "C29")
 					(unit 1)
 				)
@@
 		(dnp no)
 		(fields_autoplaced yes)
-		(property "Reference" "U?"
+		(property "Reference" "U1"
 			(at 61.8841 41.91 0)
 			(effects
@@
 			(project "diggi_shield_2"
 				(path "/21684161-6457-4723-8fc3-25d7330779e2/4a4e12e0-86da-4c7e-aa92-3e2740ba45ee"
-					(reference "U?")
+					(reference "U1")
 					(unit 1)
 				)
@@
 		(dnp no)
 		(fields_autoplaced yes)
-		(property "Reference" "C?"
+		(property "Reference" "C33"
 			(at 233.68 38.1062 0)
 			(effects
@@
 			(project "diggi_shield_2"
 				(path "/21684161-6457-4723-8fc3-25d7330779e2/4a4e12e0-86da-4c7e-aa92-3e2740ba45ee"
-					(reference "C?")
+					(reference "C33")
 					(unit 1)
 				)
@@
 		(dnp no)
 		(fields_autoplaced yes)
-		(property "Reference" "C?"
+		(property "Reference" "C31"
 			(at 146.05 36.8362 0)
 			(effects
@@
 			(project "diggi_shield_2"
 				(path "/21684161-6457-4723-8fc3-25d7330779e2/4a4e12e0-86da-4c7e-aa92-3e2740ba45ee"
-					(reference "C?")
+					(reference "C31")
 					(unit 1)
 				)
@@
 		(dnp no)
 		(fields_autoplaced yes)
-		(property "Reference" "C?"
+		(property "Reference" "C30"
 			(at 104.14 36.8362 0)
 			(effects
@@
 			(project "diggi_shield_2"
 				(path "/21684161-6457-4723-8fc3-25d7330779e2/4a4e12e0-86da-4c7e-aa92-3e2740ba45ee"
-					(reference "C?")
+					(reference "C30")
 					(unit 1)
 				)
@@
 		(dnp no)
 		(fields_autoplaced yes)
-		(property "Reference" "U?"
+		(property "Reference" "U5"
 			(at 233.3341 41.91 0)
 			(effects
@@
 			(project "diggi_shield_2"
 				(path "/21684161-6457-4723-8fc3-25d7330779e2/4a4e12e0-86da-4c7e-aa92-3e2740ba45ee"
-					(reference "U?")
+					(reference "U5")
 					(unit 1)
 				)
@@
 		(dnp no)
 		(fields_autoplaced yes)
-		(property "Reference" "U?"
+		(property "Reference" "U4"
 			(at 188.8841 41.91 0)
 			(effects
@@
 			(project "diggi_shield_2"
 				(path "/21684161-6457-4723-8fc3-25d7330779e2/4a4e12e0-86da-4c7e-aa92-3e2740ba45ee"
-					(reference "U?")
+					(reference "U4")
 					(unit 1)
 				)
@@
 		(dnp no)
 		(fields_autoplaced yes)
-		(property "Reference" "U?"
+		(property "Reference" "U3"
 			(at 145.7041 41.91 0)
 			(effects
@@
 			(project "diggi_shield_2"
 				(path "/21684161-6457-4723-8fc3-25d7330779e2/4a4e12e0-86da-4c7e-aa92-3e2740ba45ee"
-					(reference "U?")
+					(reference "U3")
 					(unit 1)
 				)
@@
 		(dnp no)
 		(fields_autoplaced yes)
-		(property "Reference" "C?"
+		(property "Reference" "C32"
 			(at 189.23 36.8362 0)
 			(effects
@@
 			(project "diggi_shield_2"
 				(path "/21684161-6457-4723-8fc3-25d7330779e2/4a4e12e0-86da-4c7e-aa92-3e2740ba45ee"
-					(reference "C?")
-					(unit 1)
-				)
+					(reference "C32")
+					(unit 1)
+				)

Commit message: Cleaned up ERC errors
Connections:
- net +3.3V: now also U1.16 (VCC), U2.16 (VCC), U3.16 (VCC), U4.16 (VCC), U5.16 (VCC)
- net GND: now also C29.2, C30.2, C31.2, C32.2, C33.2, U3.8 (GND), U4.8 (GND), U5.8 (GND)
- no-connect marks 1 -> 7
Other:
- moved on the sheet: C29, C30, C31, C32, C33

Commit message: Solve all warnings
Changed lines of the file:
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@@
-	)
-	(junction
-		(at 130.81 80.01)
-		(diameter 0)
-		(color 0 0 0 0)
 	)
 	(junction
@@
 	)
 	(junction
-		(at 173.99 80.01)
-		(diameter 0)
-		(color 0 0 0 0)
-	)
-	(junction
 		(at 101.6 38.1)
 		(diameter 0)
@@
 	(wire
 		(pts
+			(xy 236.22 39.37) (xy 245.11 39.37)
+		)
+		(stroke
+			(width 0)
+			(type default)
+		)
+	)
+	(wire
+		(pts
+			(xy 215.9 54.61) (xy 218.44 54.61)
+		)
+		(stroke
+			(width 0)
+			(type default)
+		)
+	)
+	(wire
+		(pts
+			(xy 171.45 62.23) (xy 173.99 62.23)
+		)
+		(stroke
+			(width 0)
+			(type default)
+		)
+	)
+	(wire
+		(pts
+			(xy 143.51 35.56) (xy 143.51 38.1)
+		)
+		(stroke
+			(width 0)
+			(type default)
+		)
+	)
+	(wire
+		(pts
+			(xy 128.27 69.85) (xy 130.81 69.85)
+		)
+		(stroke
+			(width 0)
+			(type default)
+		)
+	)
+	(wire
+		(pts
+			(xy 101.6 38.1) (xy 101.6 41.91)
+		)
+		(stroke
+			(width 0)
+			(type default)
+		)
+	)
+	(wire
+		(pts
+			(xy 186.69 35.56) (xy 186.69 38.1)
+		)
+		(stroke
+			(width 0)
+			(type default)
+		)
+	)
+	(wire
+		(pts
+			(xy 171.45 54.61) (xy 173.99 54.61)
+		)
+		(stroke
+			(width 0)
+			(type default)
+		)
+	)
+	(wire
+		(pts
+			(xy 218.44 82.55) (xy 218.44 87.63)
+		)
+		(stroke
+			(width 0)
+			(type default)
+		)
+	)
+	(wire
+		(pts
+			(xy 128.27 54.61) (xy 130.81 54.61)
+		)
+		(stroke
+			(width 0)
+			(type default)
+		)
+	)
+	(wire
+		(pts
+			(xy 46.99 82.55) (xy 46.99 87.63)
+		)
+		(stroke
+			(width 0)
+			(type default)
+		)
+	)
+	(wire
+		(pts
+			(xy 87.63 80.01) (xy 88.9 80.01)
+		)
+		(stroke
+			(width 0)
+			(type default)
+		)
+	)
+	(wire
+		(pts
+			(xy 186.69 90.17) (xy 186.69 91.44)
+		)
+		(stroke
+			(width 0)
+			(type default)
+		)
+	)
+	(wire
+		(pts
 			(xy 172.72 80.01) (xy 173.99 80.01)
 		)
@@
 	(wire
 		(pts
-			(xy 236.22 39.37) (xy 245.11 39.37)
-		)
-		(stroke
-			(width 0)
-			(type default)
-		)
-	)
-	(wire
-		(pts
-			(xy 215.9 54.61) (xy 218.44 54.61)
-		)
-		(stroke
-			(width 0)
-			(type default)
-		)
-	)
-	(wire
-		(pts
-			(xy 171.45 62.23) (xy 173.99 62.23)
-		)
-		(stroke
-			(width 0)
-			(type default)
-		)
-	)
-	(wire
-		(pts
-			(xy 143.51 35.56) (xy 143.51 38.1)
-		)
-		(stroke
-			(width 0)
-			(type default)
-		)
-	)
-	(wire
-		(pts
-			(xy 128.27 69.85) (xy 130.81 69.85)
-		)
-		(stroke
-			(width 0)
-			(type default)
-		)
-	)
-	(wire
-		(pts
-			(xy 101.6 38.1) (xy 101.6 41.91)
-		)
-		(stroke
-			(width 0)
-			(type default)
-		)
-	)
-	(wire
-		(pts
-			(xy 186.69 35.56) (xy 186.69 38.1)
-		)
-		(stroke
-			(width 0)
-			(type default)
-		)
-	)
-	(wire
-		(pts
-			(xy 171.45 54.61) (xy 173.99 54.61)
-		)
-		(stroke
-			(width 0)
-			(type default)
-		)
-	)
-	(wire
-		(pts
-			(xy 218.44 82.55) (xy 218.44 87.63)
-		)
-		(stroke
-			(width 0)
-			(type default)
-		)
-	)
-	(wire
-		(pts
-			(xy 128.27 54.61) (xy 130.81 54.61)
-		)
-		(stroke
-			(width 0)
-			(type default)
-		)
-	)
-	(wire
-		(pts
-			(xy 46.99 82.55) (xy 46.99 87.63)
-		)
-		(stroke
-			(width 0)
-			(type default)
-		)
-	)
-	(wire
-		(pts
-			(xy 87.63 80.01) (xy 88.9 80.01)
-		)
-		(stroke
-			(width 0)
-			(type default)
-		)
-	)
-	(wire
-		(pts
-			(xy 186.69 90.17) (xy 186.69 91.44)
-		)
-		(stroke
-			(width 0)
-			(type default)
-		)
-	)
-	(wire
-		(pts
 			(xy 171.45 57.15) (xy 173.99 57.15)
 		)
@@
 	(wire
 		(pts
+			(xy 129.54 80.01) (xy 130.81 80.01)
+		)
+		(stroke
+			(width 0)
+			(type default)
+		)
+	)
+	(wire
+		(pts
 			(xy 148.59 38.1) (xy 157.48 38.1)
 		)
@@
 	(wire
 		(pts
-			(xy 129.54 80.01) (xy 130.81 80.01)
-		)
-		(stroke
-			(width 0)
-			(type default)
-		)
-	)
-	(wire
-		(pts
 			(xy 215.9 57.15) (xy 218.44 57.15)
 		)
@@
 	(wire
 		(pts
-			(xy 130.81 80.01) (xy 132.08 80.01)
-		)
-		(stroke
-			(width 0)
-			(type default)
-		)
-	)
-	(wire
-		(pts
 			(xy 44.45 54.61) (xy 46.99 54.61)
 		)
@@
 		)
 		(stroke
-			(width 0)
-			(type default)
-		)
-	)
-	(wire
-		(pts
-			(xy 173.99 80.01) (xy 175.26 80.01)
-		)
-		(stroke

Commit message: Added jack symbols and footprints also footprints for ics and caps
Parts:
- C29, C30, C31, C32, C33: footprint (none) -> Capacitor_SMD:C_0603_1608Metric
- U1, U2, U3, U4, U5: footprint (none) -> diggi_footprints:SOP65P640X120-16
Changed lines of the file:
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@@
 			)
 		)
-		(property "Footprint" ""
+		(property "Footprint" "diggi_footprints:SOP65P640X120-16"
 			(at 101.6 64.77 0)
 			(effects
@@
 			)
 		)
-		(property "Footprint" ""
+		(property "Footprint" "Capacitor_SMD:C_0603_1608Metric"
 			(at 62.23 38.1 0)
 			(effects
@@
 			)
 		)
-		(property "Footprint" ""
+		(property "Footprint" "diggi_footprints:SOP65P640X120-16"
 			(at 59.69 64.77 0)
 			(effects
@@
 			)
 		)
-		(property "Footprint" ""
+		(property "Footprint" "Capacitor_SMD:C_0603_1608Metric"
 			(at 233.68 39.37 0)
 			(effects
@@
 			)
 		)
-		(property "Footprint" ""
+		(property "Footprint" "Capacitor_SMD:C_0603_1608Metric"
 			(at 146.05 38.1 0)
 			(effects
@@
 			)
 		)
-		(property "Footprint" ""
+		(property "Footprint" "Capacitor_SMD:C_0603_1608Metric"
 			(at 104.14 38.1 0)
 			(effects
@@
 			)
 		)
-		(property "Footprint" ""
+		(property "Footprint" "diggi_footprints:SOP65P640X120-16"
 			(at 231.14 64.77 0)
 			(effects
@@
 			)
 		)
-		(property "Footprint" ""
+		(property "Footprint" "diggi_footprints:SOP65P640X120-16"
 			(at 186.69 64.77 0)
 			(effects
@@
 			)
 		)
-		(property "Footprint" ""
+		(property "Footprint" "diggi_footprints:SOP65P640X120-16"
 			(at 143.51 64.77 0)
 			(effects
@@
 			)
 		)
-		(property "Footprint" ""
+		(property "Footprint" "Capacitor_SMD:C_0603_1608Metric"
 			(at 189.23 38.1 0)
 			(effects
